File: kicad_usb_co2.sch (KiCad schematic (older format))
At the start: 10 parts, among them SW1 SW_Push, SW2 SW_Push, U1 MH-Z14A, U2 SeeeduinoXIAO

Commit message: LEDを削除、タクトスイッチからトグルスイッチに変更
Parts:
- removed D1, D2: LED, LED_THT:LED_D5.0mm, symbol Device:LED
- removed R3, R4: R, Resistor_THT:R_Axial_DIN0207_L6.3mm_D2.5mm_P10.16mm_Horizontal, symbol Device:R
- removed SW1, SW2: SW_Push, Button_Switch_THT:SW_PUSH_6mm, symbol Switch:SW_Push
- removed U2: SeeeduinoXIAO, Seeeduino XIAO:Seeeduino XIAO-MOUDLE14P-2.54-21X17.8MM, symbol Seeeduino~XIAO:SeeeduinoXIAO
- added SW1, SW2: SW_SPDT, Mylib:SW_SLIDE_sengoku, symbol Switch:SW_SPDT
- added U2: SeeeduinoXIAO, Seeeduino XIAO:Seeeduino XIAO-MOUDLE14P-2.54-21X17.8MM, symbol Seeeduino_XIAO:SeeeduinoXIAO
Connections:
- wire segments 22 -> 20
- no-connect marks 28 -> 32
Changed lines of the file:
@@
 	4550 2550 5100 2550
-$Comp
-L Device:LED D2
-U 1 1 5EED1A13
-P 2700 1950
-F 0 "D2" V 2739 1833 50  0000 R CNN
-F 1 "LED" V 2648 1833 50  0000 R CNN
-F 2 "LED_THT:LED_D5.0mm" H 2700 1950 50  0001 C CNN
-F 3 "~" H 2700 1950 50  0001 C CNN
-	1    2700 1950
-	0    -1   -1   0
-$EndComp
-$Comp
-L Device:LED D1
-U 1 1 5EED31C5
-P 2350 2100
-F 0 "D1" V 2389 1983 50  0000 R CNN
-F 1 "LED" V 2298 1983 50  0000 R CNN
-F 2 "LED_THT:LED_D5.0mm" H 2350 2100 50  0001 C CNN
-F 3 "~" H 2350 2100 50  0001 C CNN
-	1    2350 2100
-	0    -1   -1   0
-$EndComp
-$Comp
-L Switch:SW_Push SW2
-U 1 1 5EED38F6
-P 1750 2450
-F 0 "SW2" V 1704 2598 50  0000 L CNN
-F 1 "SW_Push" V 1795 2598 50  0000 L CNN
-F 2 "Button_Switch_THT:SW_PUSH_6mm" H 1750 2650 50  0001 C CNN
-F 3 "~" H 1750 2650 50  0001 C CNN
-	1    1750 2450
-	0    1    1    0
-$EndComp
-$Comp
-L Switch:SW_Push SW1
-U 1 1 5EEDC783
-P 1200 2600
-F 0 "SW1" V 1154 2748 50  0000 L CNN
-F 1 "SW_Push" V 1245 2748 50  0000 L CNN
-F 2 "Button_Switch_THT:SW_PUSH_6mm" H 1200 2800 50  0001 C CNN
-F 3 "~" H 1200 2800 50  0001 C CNN
-	1    1200 2600
-	0    1    1    0
-$EndComp
 $Comp
 L Device:R R1
@@
 	2800 4350 2900 4350
 $Comp
-L Seeeduino~XIAO:SeeeduinoXIAO U2
-U 1 1 5EECAB2A
-P 3750 2850
-F 0 "U2" H 3725 1911 50  0000 C CNN
-F 1 "SeeeduinoXIAO" H 3725 1820 50  0000 C CNN
-F 2 "Seeeduino XIAO:Seeeduino XIAO-MOUDLE14P-2.54-21X17.8MM" H 3400 3050 50  0001 C CNN
-F 3 "" H 3400 3050 50  0001 C CNN
-	1    3750 2850
-	1    0    0    -1
-$EndComp
-$Comp
-L Device:R R3
-U 1 1 5EEEDAFB
-P 2350 2400
-F 0 "R3" H 2420 2446 50  0000 L CNN
-F 1 "R" H 2420 2355 50  0000 L CNN
-F 2 "Resistor_THT:R_Axial_DIN0207_L6.3mm_D2.5mm_P10.16mm_Horizontal" V 2280 2400 50  0001 C CNN
-F 3 "~" H 2350 2400 50  0001 C CNN
-	1    2350 2400
-	1    0    0    -1
-$EndComp
-$Comp
-L Device:R R4
-U 1 1 5EEEE419
-P 2700 2250
-F 0 "R4" H 2770 2296 50  0000 L CNN
-F 1 "R" H 2770 2205 50  0000 L CNN
-F 2 "Resistor_THT:R_Axial_DIN0207_L6.3mm_D2.5mm_P10.16mm_Horizontal" V 2630 2250 50  0001 C CNN
-F 3 "~" H 2700 2250 50  0001 C CNN
-	1    2700 2250
-	1    0    0    -1
-$EndComp
-$Comp
 L power:+3V3 #PWR0108
 U 1 1 5EEEF936
-P 1200 2400
-F 0 "#PWR0108" H 1200 2250 50  0001 C CNN
-F 1 "+3V3" H 1215 2573 50  0000 C CNN
-F 2 "" H 1200 2400 50  0001 C CNN
-F 3 "" H 1200 2400 50  0001 C CNN
-	1    1200 2400
+P 1100 2400
+F 0 "#PWR0108" H 1100 2250 50  0001 C CNN
+F 1 "+3V3" H 1115 2573 50  0000 C CNN
+F 2 "" H 1100 2400 50  0001 C CNN
+F 3 "" H 1100 2400 50  0001 C CNN
+	1    1100 2400
 	1    0    0    -1
 $EndComp
@@
 L power:+3V3 #PWR0109
 U 1 1 5EEEFFBA
-P 1750 2250
-F 0 "#PWR0109" H 1750 2100 50  0001 C CNN
-F 1 "+3V3" H 1765 2423 50  0000 C CNN
-F 2 "" H 1750 2250 50  0001 C CNN
-F 3 "" H 1750 2250 50  0001 C CNN
-	1    1750 2250
-	1    0    0    -1
-$EndComp
-$Comp
-L power:+3V3 #PWR0110
-U 1 1 5EEF067E
-P 2350 1950
-F 0 "#PWR0110" H 2350 1800 50  0001 C CNN
-F 1 "+3V3" H 2365 2123 50  0000 C CNN
-F 2 "" H 2350 1950 50  0001 C CNN
-F 3 "" H 2350 1950 50  0001 C CNN
-	1    2350 1950
-	1    0    0    -1
-$EndComp
-$Comp
-L power:+3V3 #PWR0111
-U 1 1 5EEF0CB5
-P 2700 1800
-F 0 "#PWR0111" H 2700 1650 50  0001 C CNN
-F 1 "+3V3" H 2715 1973 50  0000 C CNN
-F 2 "" H 2700 1800 50  0001 C CNN
-F 3 "" H 2700 1800 50  0001 C CNN
-	1    2700 1800
-	1    0    0    -1
-$EndComp
-Wire Wire Line
-	2900 2400 2700 2400
-Wire Wire Line
-	2900 2550 2350 2550
+P 1650 2250
+F 0 "#PWR0109" H 1650 2100 50  0001 C CNN
+F 1 "+3V3" H 1665 2423 50  0000 C CNN
+F 2 "" H 1650 2250 50  0001 C CNN
+F 3 "" H 1650 2250 50  0001 C CNN
+	1    1650 2250
+	1    0    0    -1
+$EndComp
 Wire Wire Line
 	1750 2650 1750 2700
@@
 Wire Wire Line
 	4750 2700 4550 2700
+$Comp
+L Seeeduino_XIAO:SeeeduinoXIAO U2
+U 1 1 5F3D41B4
+P 3750 2850
+F 0 "U2" H 3725 1911 50  0000 C CNN
+F 1 "SeeeduinoXIAO" H 3725 1820 50  0000 C CNN
+F 2 "Seeeduino XIAO:Seeeduino XIAO-MOUDLE14P-2.54-21X17.8MM" H 3400 3050 50  0001 C CNN
+F 3 "" H 3400 3050 50  0001 C CNN
+	1    3750 2850
+	1    0    0    -1
+$EndComp
+$Comp
+L Switch:SW_SPDT SW2
+U 1 1 5F3D6A6E
+P 1650 2450
+F 0 "SW2" V 1604 2598 50  0000 L CNN
+F 1 "SW_SPDT" V 1695 2598 50  0000 L CNN
+F 2 "Mylib:SW_SLIDE_sengoku" H 1650 2450 50  0001 C CNN
+F 3 "~" H 1650 2450 50  0001 C CNN
+	1    1650 2450
+	0    1    1    0
+$EndComp
+$Comp
+L Switch:SW_SPDT SW1
+U 1 1 5F3D76FF
+P 1100 2600
+F 0 "SW1" V 1054 2748 50  0000 L CNN
+F 1 "SW_SPDT" V 1145 2748 50  0000 L CNN
+F 2 "Mylib:SW_SLIDE_sengoku" H 1100 2600 50  0001 C CNN
+F 3 "~" H 1100 2600 50  0001 C CNN
+	1    1100 2600
+	0    1    1    0
+$EndComp
+NoConn ~ 2900 2400
+NoConn ~ 2900 2550
+NoConn ~ 1550 2650
+NoConn ~ 1000 2800
 $EndSCHEMATC
