File: kicad_mhz19b/kicad_usb_co2.sch (KiCad schematic (older format))
At the start: 6 parts, among them SW1 SW_SPDT, SW2 SW_SPDT, U1 MH-Z14A, U2 SeeeduinoXIAO

Commit message: MH-Z14A→MH-Z19Bへ置き換え、ERC OK、フットプリント関連付けはまだ
Parts:
- removed U1: MH-Z14A, MH-Z14A:MH-Z14A, symbol My_lib:MH-Z14A
- added U1: MH-Z19B, symbol MH-Z19B:MH-Z19B
Connections:
- net +3V3: now also U1.9 (Vin)
- net GND: now also U1.8 (GND)
- net at U2.6 (PA9_A5_D5_SCL): now also U1.4 (Rx)
- net at U2.7 (PB08_A6_D6_TX): now also U1.3 (Tx)
- no-connect marks 32 -> 19
Changed lines of the file:
@@
 $EndComp
 Wire Wire Line
-	2900 4450 2700 4450
+	2900 4650 2700 4650
 Wire Wire Line
-	2800 4350 2900 4350
+	2800 4500 2900 4500
 $Comp
 L power:+3V3 #PWR0108
@@
 	2900 3300 2800 3300
 Wire Wire Line
-	2800 3300 2800 4350
-Wire Wire Line
 	2900 3150 2700 3150
-Wire Wire Line
-	2700 3150 2700 4450
 NoConn ~ 4550 2400
 NoConn ~ 4550 3000
@@
 	1    0    0    -1
 $EndComp
-NoConn ~ 2250 -1350
-$Comp
-L My_lib:MH-Z14A U1
-U 1 1 5EEF3B31
-P 2900 4350
-F 0 "U1" H 3475 4615 50  0000 C CNN
-F 1 "MH-Z14A" H 3475 4524 50  0000 C CNN
-F 2 "MH-Z14A:MH-Z14A" H 3050 4500 50  0001 C CNN
-F 3 "" H 3050 4500 50  0001 C CNN
-	1    2900 4350
-	1    0    0    -1
-$EndComp
 $Comp
 L power:+3V3 #PWR0104
 U 1 1 5EF094D8
-P 2550 4550
-F 0 "#PWR0104" H 2550 4400 50  0001 C CNN
-F 1 "+3V3" H 2565 4723 50  0000 C CNN
-F 2 "" H 2550 4550 50  0001 C CNN
-F 3 "" H 2550 4550 50  0001 C CNN
-	1    2550 4550
+P 3850 4800
+F 0 "#PWR0104" H 3850 4650 50  0001 C CNN
+F 1 "+3V3" H 3865 4973 50  0000 C CNN
+F 2 "" H 3850 4800 50  0001 C CNN
+F 3 "" H 3850 4800 50  0001 C CNN
+	1    3850 4800
 	1    0    0    -1
 $EndComp
@@
 L power:GND #PWR0107
 U 1 1 5EF09D7E
-P 2550 4650
-F 0 "#PWR0107" H 2550 4400 50  0001 C CNN
-F 1 "GND" H 2555 4477 50  0000 C CNN
-F 2 "" H 2550 4650 50  0001 C CNN
-F 3 "" H 2550 4650 50  0001 C CNN
-	1    2550 4650
+P 3750 4900
+F 0 "#PWR0107" H 3750 4650 50  0001 C CNN
+F 1 "GND" H 3755 4727 50  0000 C CNN
+F 2 "" H 3750 4900 50  0001 C CNN
+F 3 "" H 3750 4900 50  0001 C CNN
+	1    3750 4900
 	1    0    0    -1
 $EndComp
-Wire Wire Line
-	2900 4550 2550 4550
-Wire Wire Line
-	2900 4650 2550 4650
-NoConn ~ 4050 4450
-NoConn ~ 4050 4550
-NoConn ~ 4050 4650
-NoConn ~ 4050 4750
-NoConn ~ 4050 4850
-NoConn ~ 4050 4950
-NoConn ~ 4050 5050
-NoConn ~ 4050 5150
-NoConn ~ 4050 5250
-NoConn ~ 2900 5250
-NoConn ~ 2900 5150
-NoConn ~ 2900 5050
-NoConn ~ 2900 4950
-NoConn ~ 2900 4850
-NoConn ~ 2900 4750
 NoConn ~ 4550 2850
 $Comp
@@
 NoConn ~ 1550 2650
 NoConn ~ 1000 2800
+$Comp
+L MH-Z19B:MH-Z19B U1
+U 1 1 5F7ADA5F
+P 2900 4200
+F 0 "U1" H 3275 4425 50  0000 C CNN
+F 1 "MH-Z19B" H 3275 4334 50  0000 C CNN
+F 2 "" H 3000 4300 50  0001 C CNN
+F 3 "" H 3000 4300 50  0001 C CNN
+	1    2900 4200
+	1    0    0    -1
+$EndComp
+Wire Wire Line
+	2700 3150 2700 4650
+Wire Wire Line
+	3850 4800 3650 4800
+Wire Wire Line
+	3650 4650 3750 4650
+Wire Wire Line
+	3750 4650 3750 4900
+NoConn ~ 3650 4350
+NoConn ~ 2900 4800
+NoConn ~ 2900 4200
+Wire Wire Line
+	2800 3300 2800 4500
 $EndSCHEMATC

Commit message: スキーマ引き直した
Parts:
- U1: footprint (none) -> MH-Z19B:MH-Z19B
Connections:
- wire segments 21 -> 34
- no-connect marks 19 -> 13
Other:
- moved on the sheet: U1
Changed lines of the file:
@@
 	1    0    0    -1
 $EndComp
-Wire Wire Line
-	2900 4650 2700 4650
-Wire Wire Line
-	2800 4500 2900 4500
 $Comp
 L power:+3V3 #PWR0108
@@
 Wire Wire Line
 	1200 2850 1200 3050
-Wire Wire Line
-	2900 3300 2800 3300
-Wire Wire Line
-	2900 3150 2700 3150
 NoConn ~ 4550 2400
 NoConn ~ 4550 3000
-NoConn ~ 4550 3150
-NoConn ~ 4550 3300
-NoConn ~ 2900 3000
 NoConn ~ 4000 1950
 NoConn ~ 3850 1950
@@
 L power:+3V3 #PWR0104
 U 1 1 5EF094D8
-P 3850 4800
-F 0 "#PWR0104" H 3850 4650 50  0001 C CNN
-F 1 "+3V3" H 3865 4973 50  0000 C CNN
-F 2 "" H 3850 4800 50  0001 C CNN
-F 3 "" H 3850 4800 50  0001 C CNN
-	1    3850 4800
+P 4100 4900
+F 0 "#PWR0104" H 4100 4750 50  0001 C CNN
+F 1 "+3V3" H 4115 5073 50  0000 C CNN
+F 2 "" H 4100 4900 50  0001 C CNN
+F 3 "" H 4100 4900 50  0001 C CNN
+	1    4100 4900
 	1    0    0    -1
 $EndComp
@@
 L power:GND #PWR0107
 U 1 1 5EF09D7E
-P 3750 4900
-F 0 "#PWR0107" H 3750 4650 50  0001 C CNN
-F 1 "GND" H 3755 4727 50  0000 C CNN
-F 2 "" H 3750 4900 50  0001 C CNN
-F 3 "" H 3750 4900 50  0001 C CNN
-	1    3750 4900
+P 4000 5000
+F 0 "#PWR0107" H 4000 4750 50  0001 C CNN
+F 1 "GND" H 4005 4827 50  0000 C CNN
+F 2 "" H 4000 5000 50  0001 C CNN
+F 3 "" H 4000 5000 50  0001 C CNN
+	1    4000 5000
 	1    0    0    -1
 $EndComp
@@
 NoConn ~ 1550 2650
 NoConn ~ 1000 2800
+Wire Wire Line
+	4000 4750 4000 5000
+Wire Wire Line
+	4100 4900 3950 4900
+Wire Wire Line
+	3900 4750 3950 4750
 $Comp
 L MH-Z19B:MH-Z19B U1
 U 1 1 5F7ADA5F
-P 2900 4200
-F 0 "U1" H 3275 4425 50  0000 C CNN
-F 1 "MH-Z19B" H 3275 4334 50  0000 C CNN
-F 2 "" H 3000 4300 50  0001 C CNN
-F 3 "" H 3000 4300 50  0001 C CNN
-	1    2900 4200
-	1    0    0    -1
-$EndComp
-Wire Wire Line
-	2700 3150 2700 4650
-Wire Wire Line
-	3850 4800 3650 4800
-Wire Wire Line
-	3650 4650 3750 4650
-Wire Wire Line
-	3750 4650 3750 4900
-NoConn ~ 3650 4350
-NoConn ~ 2900 4800
-NoConn ~ 2900 4200
-Wire Wire Line
-	2800 3300 2800 4500
+P 3200 4300
+F 0 "U1" H 3575 4525 50  0000 C CNN
+F 1 "MH-Z19B" H 3575 4434 50  0000 C CNN
+F 2 "MH-Z19B:MH-Z19B" H 3300 4400 50  0001 C CNN
+F 3 "" H 3300 4400 50  0001 C CNN
+	1    3200 4300
+	1    0    0    -1
+$EndComp
+Connection ~ 3950 4750
+Wire Wire Line
+	3950 4750 4000 4750
+Connection ~ 3950 4900
+Wire Wire Line
+	3950 4900 3900 4900
+Wire Wire Line
+	4750 3950 3150 3950
+Wire Wire Line
+	3150 3950 3150 4300
+Wire Wire Line
+	3150 4300 3200 4300
+Wire Wire Line
+	4650 4450 3950 4450
+Wire Wire Line
+	2800 4900 3200 4900
+Wire Wire Line
+	2600 4600 3200 4600
+Wire Wire Line
+	2700 4750 3200 4750
+Wire Wire Line
+	2900 3000 2800 3000
+Wire Wire Line
+	2800 3000 2800 4900
+Wire Wire Line
+	2900 3150 2700 3150
+Wire Wire Line
+	2700 3150 2700 4750
+Wire Wire Line
+	2900 3300 2600 3300
+Wire Wire Line
+	2600 3300 2600 4600
+Wire Wire Line
+	4550 3150 4650 3150
+Wire Wire Line
+	4650 3150 4650 4450
+Wire Wire Line
+	4550 3300 4750 3300
+Wire Wire Line
+	4750 3300 4750 3950
 $EndSCHEMATC

Commit message: センサの電源を3.3Vから5Vに変えた
Connections:
- net labels added: +5V
- net labels removed: +3V3
Changed lines of the file:
@@
-	1    0    0    -1
-$EndComp
-$Comp
-L power:+3V3 #PWR0108
-U 1 1 5EEEF936
-P 1100 2400
-F 0 "#PWR0108" H 1100 2250 50  0001 C CNN
-F 1 "+3V3" H 1115 2573 50  0000 C CNN
-F 2 "" H 1100 2400 50  0001 C CNN
-F 3 "" H 1100 2400 50  0001 C CNN
-	1    1100 2400
-	1    0    0    -1
-$EndComp
-$Comp
-L power:+3V3 #PWR0109
-U 1 1 5EEEFFBA
-P 1650 2250
-F 0 "#PWR0109" H 1650 2100 50  0001 C CNN
-F 1 "+3V3" H 1665 2423 50  0000 C CNN
-F 2 "" H 1650 2250 50  0001 C CNN
-F 3 "" H 1650 2250 50  0001 C CNN
-	1    1650 2250
 	1    0    0    -1
 $EndComp
@@
 Wire Wire Line
 	1200 2850 1200 3050
-NoConn ~ 4550 2400
+NoConn ~ 4550 2700
 NoConn ~ 4550 3000
 NoConn ~ 4000 1950
@@
 	1200 1300 1550 1300
 $Comp
-L power:+3V3 #PWR0101
-U 1 1 5EECA17D
-P 1550 1100
-F 0 "#PWR0101" H 1550 950 50  0001 C CNN
-F 1 "+3V3" H 1565 1273 50  0000 C CNN
-F 2 "" H 1550 1100 50  0001 C CNN
-F 3 "" H 1550 1100 50  0001 C CNN
-	1    1550 1100
-	1    0    0    -1
-$EndComp
-$Comp
-L power:+3V3 #PWR0104
-U 1 1 5EF094D8
-P 4100 4900
-F 0 "#PWR0104" H 4100 4750 50  0001 C CNN
-F 1 "+3V3" H 4115 5073 50  0000 C CNN
-F 2 "" H 4100 4900 50  0001 C CNN
-F 3 "" H 4100 4900 50  0001 C CNN
-	1    4100 4900
-	1    0    0    -1
-$EndComp
-$Comp
 L power:GND #PWR0107
 U 1 1 5EF09D7E
@@
 $EndComp
 NoConn ~ 4550 2850
-$Comp
-L power:+3V3 #PWR0112
-U 1 1 5EF136B9
-P 4750 2700
-F 0 "#PWR0112" H 4750 2550 50  0001 C CNN
-F 1 "+3V3" H 4765 2873 50  0000 C CNN
-F 2 "" H 4750 2700 50  0001 C CNN
-F 3 "" H 4750 2700 50  0001 C CNN
-	1    4750 2700
-	1    0    0    -1
-$EndComp
-Wire Wire Line
-	4750 2700 4550 2700
+Wire Wire Line
+	4750 2400 4550 2400
 $Comp
 L Seeeduino_XIAO:SeeeduinoXIAO U2
@@
 	0    1    1    0
 $EndComp
+NoConn ~ 2900 2400
+NoConn ~ 2900 2550
+NoConn ~ 1550 2650
+NoConn ~ 1000 2800
+Wire Wire Line
+	4000 4750 4000 5000
+Wire Wire Line
+	4100 4900 3950 4900
+Wire Wire Line
+	3900 4750 3950 4750
+$Comp
+L MH-Z19B:MH-Z19B U1
+U 1 1 5F7ADA5F
+P 3200 4300
+F 0 "U1" H 3575 4525 50  0000 C CNN
+F 1 "MH-Z19B" H 3575 4434 50  0000 C CNN
+F 2 "MH-Z19B:MH-Z19B" H 3300 4400 50  0001 C CNN
+F 3 "" H 3300 4400 50  0001 C CNN
+	1    3200 4300
+	1    0    0    -1
+$EndComp
+Connection ~ 3950 4750
+Wire Wire Line
+	3950 4750 4000 4750
+Connection ~ 3950 4900
+Wire Wire Line
+	3950 4900 3900 4900
+Wire Wire Line
+	4750 3950 3150 3950
+Wire Wire Line
+	3150 3950 3150 4300
+Wire Wire Line
+	3150 4300 3200 4300
+Wire Wire Line
+	4650 4450 3950 4450
+Wire Wire Line
+	2800 4900 3200 4900
+Wire Wire Line
+	2600 4600 3200 4600
+Wire Wire Line
+	2700 4750 3200 4750
+Wire Wire Line
+	2900 3000 2800 3000
+Wire Wire Line
+	2800 3000 2800 4900
+Wire Wire Line
+	2900 3150 2700 3150
+Wire Wire Line
+	2700 3150 2700 4750
+Wire Wire Line
+	2900 3300 2600 3300
+Wire Wire Line
+	2600 3300 2600 4600
+Wire Wire Line
+	4550 3150 4650 3150
+Wire Wire Line
+	4650 3150 4650 4450
+Wire Wire Line
+	4550 3300 4750 3300
+Wire Wire Line
+	4750 3300 4750 3950
+$Comp
+L power:+5V #PWR01
+U 1 1 5F8A276C
+P 1550 1100
+F 0 "#PWR01" H 1550 950 50  0001 C CNN
+F 1 "+5V" H 1565 1273 50  0000 C CNN
+F 2 "" H 1550 1100 50  0001 C CNN
+F 3 "" H 1550 1100 50  0001 C CNN
+	1    1550 1100
+	1    0    0    -1
+$EndComp
+$Comp
+L power:+5V #PWR02
+U 1 1 5F8A2F84
+P 4750 2400
+F 0 "#PWR02" H 4750 2250 50  0001 C CNN
+F 1 "+5V" H 4765 2573 50  0000 C CNN
+F 2 "" H 4750 2400 50  0001 C CNN
+F 3 "" H 4750 2400 50  0001 C CNN
+	1    4750 2400
+	1    0    0    -1
+$EndComp
 $Comp
 L Switch:SW_SPDT SW1
@@
 	0    1    1    0
 $EndComp
-NoConn ~ 2900 2400
-NoConn ~ 2900 2550
-NoConn ~ 1550 2650
-NoConn ~ 1000 2800
-Wire Wire Line
-	4000 4750 4000 5000
-Wire Wire Line
-	4100 4900 3950 4900
-Wire Wire Line
-	3900 4750 3950 4750
-$Comp
-L MH-Z19B:MH-Z19B U1
-U 1 1 5F7ADA5F
-P 3200 4300
-F 0 "U1" H 3575 4525 50  0000 C CNN
-F 1 "MH-Z19B" H 3575 4434 50  0000 C CNN
-F 2 "MH-Z19B:MH-Z19B" H 3300 4400 50  0001 C CNN
-F 3 "" H 3300 4400 50  0001 C CNN
-	1    3200 4300
-	1    0    0    -1
-$EndComp
-Connection ~ 3950 4750
-Wire Wire Line
-	3950 4750 4000 4750
-Connection ~ 3950 4900
-Wire Wire Line
-	3950 4900 3900 4900
-Wire Wire Line
-	4750 3950 3150 3950
-Wire Wire Line
-	3150 3950 3150 4300
-Wire Wire Line
-	3150 4300 3200 4300
-Wire Wire Line
-	4650 4450 3950 4450
-Wire Wire Line
-	2800 4900 3200 4900
-Wire Wire Line
-	2600 4600 3200 4600
-Wire Wire Line
-	2700 4750 3200 4750
-Wire Wire Line
-	2900 3000 2800 3000
-Wire Wire Line
-	2800 3000 2800 4900
-Wire Wire Line
-	2900 3150 2700 3150
-Wire Wire Line
-	2700 3150 2700 4750
-Wire Wire Line
-	2900 3300 2600 3300
-Wire Wire Line
-	2600 3300 2600 4600
-Wire Wire Line
-	4550 3150 4650 3150
-Wire Wire Line
-	4650 3150 4650 4450
-Wire Wire Line
-	4550 3300 4750 3300
-Wire Wire Line
-	4750 3300 4750 3950
+$Comp
+L power:+5V #PWR03
+U 1 1 5F8A6AAD
+P 1100 2400
+F 0 "#PWR03" H 1100 2250 50  0001 C CNN
+F 1 "+5V" H 1115 2573 50  0000 C CNN
+F 2 "" H 1100 2400 50  0001 C CNN
+F 3 "" H 1100 2400 50  0001 C CNN
+	1    1100 2400
+	1    0    0    -1
+$EndComp
+$Comp
+L power:+5V #PWR04
+U 1 1 5F8A7015
+P 1650 2250
+F 0 "#PWR04" H 1650 2100 50  0001 C CNN
+F 1 "+5V" H 1665 2423 50  0000 C CNN
+F 2 "" H 1650 2250 50  0001 C CNN
+F 3 "" H 1650 2250 50  0001 C CNN
+	1    1650 2250
+	1    0    0    -1
+$EndComp
+$Comp
+L power:+5V #PWR05
+U 1 1 5F8A88E4
+P 4100 4900
+F 0 "#PWR05" H 4100 4750 50  0001 C CNN
+F 1 "+5V" H 4115 5073 50  0000 C CNN
+F 2 "" H 4100 4900 50  0001 C CNN
+F 3 "" H 4100 4900 50  0001 C CNN
+	1    4100 4900
+	1    0    0    -1
+$EndComp
 $EndSCHEMATC
