File: kicad_mhz19b/kicad_usb_co2.kicad_pcb (KiCad board)
At the start: 2 copper layers, 90 x 54 mm, 6 parts, among them SW1 SW_SPDT, SW2 SW_SPDT, U1 MH-Z14A, U2 SeeeduinoXIAO

Commit message: 配置配線ok DRCok
Parts:
- U1: value MH-Z14A -> MH-Z19B; footprint MH-Z14A:MH-Z14A -> MH-Z19B:MH-Z19B
- moved U1 15.3 mm to (15.2, 38.1)
Connections:
- SW1 pad 2: +3V3 -> +5V
- SW2 pad 2: +3V3 -> +5V
- U1 pad 8: Net-(U1-Pad8) -> GND
- U1 pad 9: Net-(U1-Pad9) -> +5V
- U2 pad 12: +3V3 -> Net-(U2-Pad12)
- U2 pad 14: Net-(U2-Pad14) -> +5V
- U2 pad 5: Net-(U2-Pad5) -> Net-(U1-Pad5)
- U2 pad 6: Net-(U1-Pad18) -> Net-(U1-Pad4)
- U2 pad 7: Net-(U1-Pad19) -> Net-(U1-Pad3)
- U2 pad 8: Net-(U2-Pad8) -> Net-(U1-Pad1)
- U2 pad 9: Net-(U2-Pad9) -> Net-(U1-Pad6)
Routing:
- net +3V3: track 96.3 -> 0.00 mm
- net +5V: track 0.00 -> 92.5 mm
- net Net-(U1-Pad18): track 78.8 -> 0.00 mm
- net Net-(U1-Pad19): track 76.3 -> 0.00 mm
- net GND: track 78.1 -> 7.52 mm, vias 4 -> 3
- net Net-(U1-Pad6): track 0.00 -> 64.8 mm, vias 0 -> 1
- net Net-(U1-Pad5): track 0.00 -> 37.9 mm
- net Net-(U1-Pad4): track 0.00 -> 34.3 mm
- net Net-(U1-Pad1): track 0.00 -> 33.0 mm, vias 0 -> 1
- net Net-(U1-Pad3): track 0.00 -> 30.8 mm

Commit message: バージョンがrev 0.2 のままだったので、0.1に治した
Other:
- board text added: "2020 REALGLOBE Inc rev 0.1"
- board text removed: "2020 REALGLOBE Inc rev 0.2"
Changed lines of the file:
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@@
   (gr_circle (center 2.54 2.54) (end 4.04 2.54) (layer Edge.Cuts) (width 0.05))
   (gr_arc (start 2.54 2.54) (end 2.54 0) (angle -90) (layer Edge.Cuts) (width 0.05))
-  (gr_text "2020 REALGLOBE Inc rev 0.2" (at 33.02 5.08) (layer F.SilkS)
+  (gr_text "2020 REALGLOBE Inc rev 0.1" (at 33.02 5.08) (layer F.SilkS)
     (effects (font (size 1.5 1.5) (thickness 0.3)))
   )
